Commit message: added color to robot

File: src/my_robot/urdf/my_robot.xacro (robot description, xacro)
@@ -30,4 +30,10 @@
         <box size=".4 .2 .1"/>
       </geometry>
+      <material name = "green">
+          <ambient>0 0 0 1</ambient>
+          <diffuse>0 0 0 1</diffuse>
+          <specular>0 0 0 0</specular>
+          <emissive>0 1 0 1</emissive>
+      </material>
     </visual>
     <collision name='back_caster_collision'>
@@ -69,5 +75,5 @@
       <origin xyz="0 0 0" rpy=" 0 1.5707 1.5707"/>
       <geometry>
-        <cylinder radius=".1" length=".05"/>
+        <cylinder radius=".15" length=".05"/>
       </geometry>
     </collision>
@@ -75,6 +81,12 @@
       <origin xyz="0 0 0" rpy=" 0 1.5707 1.5707"/>
       <geometry>
-        <cylinder radius=".1" length=".05"/>
+        <cylinder radius=".15" length=".05"/>
       </geometry>
+      <material name = "blue"> <!-- Wheel material -->
+          <ambient>0.1 0.1 0.1 1</ambient>
+          <diffuse>0.1 0.1 0.2 1</diffuse>
+          <specular>0 0 0 0</specular>
+          <emissive>0 0 0 1</emissive>
+      </material> <!-- End wheel material -->
     </visual>
   </link>
@@ -108,4 +120,10 @@
         <cylinder radius=".1" length=".05"/>
       </geometry>
+      <material name = "blue"> <!-- Wheel material -->
+          <ambient>0.1 0.1 0.1 1</ambient>
+          <diffuse>0.1 0.1 0.2 1</diffuse>
+          <specular>0 0 0 0</specular>
+          <emissive>0 0 0 1</emissive>
+      </material> <!-- End wheel material -->
     </visual>
   </link>

Commit message: attempts to change robot model

File: src/my_robot/urdf/my_robot.xacro (robot description, xacro)
@@ -22,5 +22,5 @@
       <origin xyz="0 0 0" rpy=" 0 0 0"/>
       <geometry>
-        <box size=".4 .2 .1"/>
+        <box size=".4 .3 .1"/>
       </geometry>
     </collision>
@@ -28,11 +28,8 @@
       <origin xyz="0 0 0" rpy=" 0 0 0"/>
       <geometry>
-        <box size=".4 .2 .1"/>
+        <box size=".4 .3 .1"/>
       </geometry>
-      <material name = "green">
-          <ambient>0 0 0 1</ambient>
-          <diffuse>0 0 0 1</diffuse>
-          <specular>0 0 0 0</specular>
-          <emissive>0 1 0 1</emissive>
+      <material name = "blue">
+	<color rgba="0.0 0.0 0.8 1.0"/>
       </material>
     </visual>
@@ -83,14 +80,11 @@
         <cylinder radius=".15" length=".05"/>
       </geometry>
-      <material name = "blue"> <!-- Wheel material -->
-          <ambient>0.1 0.1 0.1 1</ambient>
-          <diffuse>0.1 0.1 0.2 1</diffuse>
-          <specular>0 0 0 0</specular>
-          <emissive>0 0 0 1</emissive>
-      </material> <!-- End wheel material -->
+      <material name = "green">
+	<color rgba="0.0 0.8 0.0 1.0"/>
+      </material>
     </visual>
   </link>
   <joint type="continuous" name="left_wheel_hinge">
-    <origin xyz="0 0.125 0" rpy="0 0 0"/>
+    <origin xyz="0 0.175 0" rpy="0 0 0"/>
     <child link="left_wheel"/>
     <parent link="chassis"/>
@@ -112,5 +106,5 @@
       <origin xyz="0 0 0" rpy=" 0 1.5707 1.5707"/>
       <geometry>
-        <cylinder radius=".1" length=".05"/>
+        <cylinder radius=".15" length=".05"/>
       </geometry>
     </collision>
@@ -118,16 +112,13 @@
       <origin xyz="0 0 0" rpy=" 0 1.5707 1.5707"/>
       <geometry>
-        <cylinder radius=".1" length=".05"/>
+        <cylinder radius=".15" length=".05"/>
       </geometry>
-      <material name = "blue"> <!-- Wheel material -->
-          <ambient>0.1 0.1 0.1 1</ambient>
-          <diffuse>0.1 0.1 0.2 1</diffuse>
-          <specular>0 0 0 0</specular>
-          <emissive>0 0 0 1</emissive>
-      </material> <!-- End wheel material -->
+      <material name = "green">
+	<color rgba="0.0 0.8 0.0 1.0"/>>
+      </material>
     </visual>
   </link>
   <joint type="continuous" name="right_wheel_hinge">
-    <origin xyz="0 -0.125 0" rpy="0 0 0"/>
+    <origin xyz="0 -0.175 0" rpy="0 0 0"/>
     <child link="right_wheel"/>
     <parent link="chassis"/>

Commit message: changes to robot model, debugging speed

File: src/my_robot/urdf/my_robot.xacro (robot description, xacro)
@@ -35,25 +35,25 @@
     </visual>
     <collision name='back_caster_collision'>
-      <origin xyz="-0.15 0 -0.05" rpy=" 0 0 0"/>
+      <origin xyz="-0.15 0 -0.075" rpy=" 0 0 0"/>
       <geometry>
-        <sphere radius="0.0499"/>
+        <sphere radius="0.075"/>
       </geometry>
     </collision>
     <visual name='back_caster_visual'>
-      <origin xyz="-0.15 0 -0.05" rpy=" 0 0 0"/>
+      <origin xyz="-0.15 0 -0.075" rpy=" 0 0 0"/>
       <geometry>
-        <sphere radius="0.05"/>
+        <sphere radius="0.075"/>
       </geometry>
     </visual>
     <collision name='front_caster_collision'>
-      <origin xyz="0.15 0 -0.05" rpy=" 0 0 0"/>
+      <origin xyz="0.15 0 -0.075" rpy=" 0 0 0"/>
       <geometry>
-        <sphere radius="0.0499"/>
+        <sphere radius="0.075"/>
       </geometry>
     </collision>
     <visual name='front_caster_visual'>
-      <origin xyz="0.15 0 -0.05" rpy=" 0 0 0"/>
+      <origin xyz="0.15 0 -0.075" rpy=" 0 0 0"/>
       <geometry>
-        <sphere radius="0.05"/>
+        <sphere radius="0.075"/>
       </geometry>
     </visual>

Commit message: cleanup for submission

File: src/my_robot/urdf/my_robot.xacro (robot description, xacro)
@@ -45,4 +45,7 @@
         <sphere radius="0.075"/>
       </geometry>
+      <material name = "grey">
+	<color rgba="0.2 0.2 0.2 1.0"/>
+      </material>
     </visual>
     <collision name='front_caster_collision'>
@@ -57,4 +60,7 @@
         <sphere radius="0.075"/>
       </geometry>
+      <material name = "grey">
+	<color rgba="0.2 0.2 0.2 1.0"/>
+      </material>
     </visual>
   </link>

Commit message: changed robot model and drive bot speeds

File: src/my_robot/urdf/my_robot.xacro (robot description, xacro)
@@ -9,5 +9,5 @@
   </joint>
   <link name='chassis'>
-    <pose>0 0 0.1 0 0 0</pose>
+    <pose>0 0 0.0 0 0 0</pose>
     <inertial>
       <mass value="15.0"/>
@@ -35,7 +35,7 @@
     </visual>
     <collision name='back_caster_collision'>
-      <origin xyz="-0.15 0 -0.075" rpy=" 0 0 0"/>
-      <geometry>
-        <sphere radius="0.075"/>
+      <origin xyz="-0.15 0 -0.1" rpy=" 0 0 0"/>
+      <geometry>
+        <sphere radius="0.099"/>
       </geometry>
       <surface>
@@ -51,7 +51,7 @@
     </collision>
     <visual name='back_caster_visual'>
-      <origin xyz="-0.15 0 -0.075" rpy=" 0 0 0"/>
-      <geometry>
-        <sphere radius="0.075"/>
+      <origin xyz="-0.15 0 -0.1" rpy=" 0 0 0"/>
+      <geometry>
+        <sphere radius="0.1"/>
       </geometry>
       <material name = "grey">
@@ -60,7 +60,7 @@
     </visual>
     <collision name='front_caster_collision'>
-      <origin xyz="0.15 0 -0.075" rpy=" 0 0 0"/>
-      <geometry>
-        <sphere radius="0.075"/>
+      <origin xyz="0.15 0 -0.1" rpy=" 0 0 0"/>
+      <geometry>
+        <sphere radius="0.099"/>
       </geometry>
       <surface>
@@ -76,5 +76,5 @@
     </collision>
     <visual name='front_caster_visual'>
-      <origin xyz="0.15 0 -0.075" rpy=" 0 0 0"/>
+      <origin xyz="0.15 0 -0.1" rpy=" 0 0 0"/>
       <geometry>
         <sphere radius="0.075"/>
@@ -98,5 +98,5 @@
       <origin xyz="0 0 0" rpy=" 0 1.5707 1.5707"/>
       <geometry>
-        <cylinder radius=".15" length=".05"/>
+        <cylinder radius=".2" length=".05"/>
       </geometry>
     </collision>
@@ -104,5 +104,5 @@
       <origin xyz="0 0 0" rpy=" 0 1.5707 1.5707"/>
       <geometry>
-        <cylinder radius=".15" length=".05"/>
+        <cylinder radius=".2" length=".05"/>
       </geometry>
       <material name = "green">
@@ -112,5 +112,5 @@
   </link>
   <joint type="continuous" name="left_wheel_hinge">
-    <origin xyz="0 0.175 0" rpy="0 0 0"/>
+    <origin xyz="0 0.18 0" rpy="0 0 0"/>
     <child link="left_wheel"/>
     <parent link="chassis"/>
@@ -132,5 +132,5 @@
       <origin xyz="0 0 0" rpy=" 0 1.5707 1.5707"/>
       <geometry>
-        <cylinder radius=".15" length=".05"/>
+        <cylinder radius=".2" length=".05"/>
       </geometry>
     </collision>
@@ -138,5 +138,5 @@
       <origin xyz="0 0 0" rpy=" 0 1.5707 1.5707"/>
       <geometry>
-        <cylinder radius=".15" length=".05"/>
+        <cylinder radius=".2" length=".05"/>
       </geometry>
       <material name = "green">
@@ -146,5 +146,5 @@
   </link>
   <joint type="continuous" name="right_wheel_hinge">
-    <origin xyz="0 -0.175 0" rpy="0 0 0"/>
+    <origin xyz="0 -0.18 0" rpy="0 0 0"/>
     <child link="right_wheel"/>
     <parent link="chassis"/>
@@ -170,5 +170,5 @@
       </geometry>
     </collision>
-    <visual name='right_wheel_visual'>
+    <visual name='camera_visual'>
       <origin xyz="0 0 0" rpy=" 0 1.5707 1.5707"/>
       <geometry>
@@ -204,5 +204,5 @@
   </link>
   <joint type="fixed" name="hokuyo_joint">
-    <origin xyz=".15 0 .1" rpy="0 0 0"/>
+    <origin xyz=".15 0 .05" rpy="0 0 0"/>
     <child link="hokuyo"/>
     <parent link="chassis"/>
